File: ads1292_Dorokhov.sch (EAGLE design)
At the start: 61 parts, among them IC1 TPS77001, Q1 BSS84, U1 LIS344AL

Commit message: Rev.2.0
Connections:
- removed net N$29: C16.1, C2.1, R11.2, R6.1, U$1.IN1N, U$4.6
- new net N$15: C1.1, C16.2, R12.2, U$1.IN1P, U$4.6
- net ACC_X: now also U$2.6; no longer U$2.8
- net ACC_Z: now also U$2.8; no longer U$2.6
- net AGND: no longer LED1.C
- net GND: now also LED1.C
- net N$21: now also R2.1; no longer R12.1
- net N$22: now also R12.1; no longer R2.1
- net N$23: now also C16.1, C2.1, R11.2, R6.1, U$1.IN1N; no longer C1.1, C16.2, R12.2, U$1.IN1P
Other:
- note added: "Перекинул светодиодик на цифровую землю"

Commit message: REV_3.0
Connections:
- removed net N$18: R6.2, U$1.RLDINV, U$1.RLDOUT
- new net N$27: R6.2, U$1.RLDIN/RLDREF, U$1.RLDINV, U$1.RLDOUT
- net +3V3: no longer U$1.RLDIN/RLDREF
Changed lines of the file:
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@@
 <wire x1="101.6" y1="93.98" x2="101.6" y2="96.52" width="0.1524" layer="91"/>
 <pinref part="+3V6" gate="G$1" pin="+3V3"/>
-<pinref part="U$1" gate="G$1" pin="RLDIN/RLDREF"/>
 <wire x1="101.6" y1="96.52" x2="101.6" y2="109.22" width="0.1524" layer="91"/>
-<wire x1="109.22" y1="93.98" x2="109.22" y2="96.52" width="0.1524" layer="91"/>
-<wire x1="109.22" y1="96.52" x2="104.14" y2="96.52" width="0.1524" layer="91"/>
 <junction x="101.6" y="96.52"/>
 <wire x1="104.14" y1="96.52" x2="101.6" y2="96.52" width="0.1524" layer="91"/>
 <wire x1="104.14" y1="93.98" x2="104.14" y2="96.52" width="0.1524" layer="91"/>
-<junction x="104.14" y="96.52"/>
 </segment>
 <segment>
@@
 </segment>
 </net>
-<net name="N$18" class="0">
-<segment>
-<pinref part="U$1" gate="G$1" pin="RLDOUT"/>
-<pinref part="U$1" gate="G$1" pin="RLDINV"/>
-<wire x1="111.76" y1="99.06" x2="111.76" y2="93.98" width="0.1524" layer="91"/>
-<wire x1="111.76" y1="99.06" x2="106.68" y2="99.06" width="0.1524" layer="91"/>
-<wire x1="106.68" y1="99.06" x2="106.68" y2="93.98" width="0.1524" layer="91"/>
-<pinref part="R6" gate="G$1" pin="2"/>
-<wire x1="88.9" y1="99.06" x2="106.68" y2="99.06" width="0.1524" layer="91"/>
-<junction x="106.68" y="99.06"/>
-</segment>
-</net>
 <net name="N$26" class="0">
 <segment>
@@
 </segment>
 </net>
+<net name="N$27" class="0">
+<segment>
+<pinref part="U$1" gate="G$1" pin="RLDIN/RLDREF"/>
+<pinref part="U$1" gate="G$1" pin="RLDOUT"/>
+<pinref part="U$1" gate="G$1" pin="RLDINV"/>
+<wire x1="111.76" y1="99.06" x2="111.76" y2="93.98" width="0.1524" layer="91"/>
+<wire x1="111.76" y1="99.06" x2="109.22" y2="99.06" width="0.1524" layer="91"/>
+<wire x1="109.22" y1="99.06" x2="106.68" y2="99.06" width="0.1524" layer="91"/>
+<wire x1="106.68" y1="99.06" x2="106.68" y2="93.98" width="0.1524" layer="91"/>
+<pinref part="R6" gate="G$1" pin="2"/>
+<wire x1="88.9" y1="99.06" x2="106.68" y2="99.06" width="0.1524" layer="91"/>
+<junction x="106.68" y="99.06"/>
+<wire x1="109.22" y1="93.98" x2="109.22" y2="99.06" width="0.1524" layer="91"/>
+<junction x="109.22" y="99.06"/>
+</segment>
+</net>
